File: KiCad/ardCurvTracer/ardCurvTracer.kicad_sch (KiCad schematic)
At the start: 62 parts

Commit message: kicad
Parts:
- added H1, H2, H3, H4: MountingHole, MountingHole:MountingHole_3.2mm_M3, symbol Mechanical:MountingHole
- Bat1: value (none) -> Battery; footprint (none) -> My_Headers:2-pin_power_input_header_larger_pads
- C1, C2, C3, C4, DC1, DC2: value (none) -> 100n; footprint (none) -> My_Misc:C_Disc_D3.0mm_W1.6mm_P2.50mm_larg
- DC3, DC4: value (none) -> 10u; footprint (none) -> My_Misc:CP_Radial_D5.0mm_P2.00mm_larger
- J1: value (none) -> 4-pin_Serial_Connection_header; footprint (none) -> My_Headers:4-pin Serial Connection header large
- Q1, Q2, Q3: value (none) -> BC639; footprint (none) -> My_Misc:TO-92_Inline_Wide_large
- QNPN1: value (none) -> NPNDUT
- QPNP1: value (none) -> PNPDUT
- R1, R2, R3, R4, R5: value (none) -> 3k3; footprint (none) -> My_Misc:R_Axial_DIN0207_L6.3mm_D2.5mm_P10.16mm_Horizontal_larger_pads
- R10, R13, R14, R15, R9: value (none) -> 2k2; footprint (none) -> My_Misc:R_Axial_DIN0207_L6.3mm_D2.5mm_P10.16mm_Horizontal_larger_pads
- R11, R12, R27, R29, R38, R6, R7, R8: value (none) -> 33k; footprint (none) -> My_Misc:R_Axial_DIN0207_L6.3mm_D2.5mm_P10.16mm_Horizontal_larger_pads
- R16, R21, R22, R24, R34, R35, R40: value (none) -> 10k; footprint (none) -> My_Misc:R_Axial_DIN0207_L6.3mm_D2.5mm_P10.16mm_Horizontal_larger_pads
- R17, R18, R19, R20, R25: value (none) -> 47k; footprint (none) -> My_Misc:R_Axial_DIN0207_L6.3mm_D2.5mm_P10.16mm_Horizontal_larger_pads
- R26: value (none) -> 27k; footprint (none) -> My_Misc:R_Axial_DIN0207_L6.3mm_D2.5mm_P10.16mm_Horizontal_larger_pads
- R28, R36: value (none) -> 68k; footprint (none) -> My_Misc:R_Axial_DIN0207_L6.3mm_D2.5mm_P10.16mm_Horizontal_larger_pads
- R30, R33: value (none) -> 1k; footprint (none) -> My_Misc:R_Axial_DIN0207_L6.3mm_D2.5mm_P10.16mm_Horizontal_larger_pads
- R31: value (none) -> 4k7; footprint (none) -> My_Misc:R_Axial_DIN0207_L6.3mm_D2.5mm_P10.16mm_Horizontal_larger_pads
- R32, R37: value (none) -> 100R 0.25W; footprint (none) -> My_Misc:R_Axial_DIN0207_L6.3mm_D2.5mm_P10.16mm_Horizontal_larger_pads
- SW1: value (none) -> On/Off; footprint (none) -> My_Parts:2-pole switch large
- U1: value (none) -> MCP4802; footprint (none) -> My_Misc:DIP-8_W7.62mm_Socket_w_dip_packet_LongPads
- U2: value (none) -> Test socket; footprint (none) -> My_Misc:ZIF_DIP_Socket-14_W4.3_W5.08_W7.62_W10.16_W10.9_3M_214-3339-00-0602J
- U3: value (none) -> LM358; footprint (none) -> My_Misc:DIP-8_W7.62mm_Socket_w_dip_packet_LongPads
- U5: value (none) -> HT7550; footprint (none) -> Package_TO_SOT_SMD:SOT-89-3
- U6: value (none) -> HT7533; footprint (none) -> Package_TO_SOT_SMD:SOT-89-3
- UBoost1: value (none) -> Step_Up_Converter; footprint (none) -> My_Parts:6V to 12V Step Up Converter
- UMCU1: value (none) -> Arduino_Mini_Pro; footprint (none) -> My_Arduino:Arduino_Pro_Mini_vA_sides_n_A4-A7_large
- UTFT1: value (none) -> ILI9341_2.8_TFT_Touch; footprint (none) -> My_Parts:ILI9341 2.8 TFT Touch large
